Commit message: [add] scripts for simulation

File: denso_robot_descriptions/vs087_description/vs087.urdf (robot description, URDF)
Before this commit: robot vs087, 8 links, 7 joints
Joints:
- joint joint_2: origin xyz=0.030000 0.000000 0.197500 rpy=0.000000 0.000000 0.000000 -> xyz=0.030000 0.000000 0.197500 rpy=0.000000 -0.34906585 0.000000
- joint joint_3: origin xyz=0.000000 0.000000 0.445000 rpy=0.000000 0.000000 0.000000 -> xyz=0.000000 0.000000 0.445000 rpy=0.000000 1.919862175 0.000000

Commit message: [add] simulation/real controller for vs087

File: denso_robot_descriptions/vs087_description/vs087.urdf (robot description, URDF)
Before this commit: robot vs087, 8 links, 7 joints
Joints:
- joint joint_2: origin xyz=0.030000 0.000000 0.197500 rpy=0.000000 -0.34906585 0.000000 -> xyz=0.030000 0.000000 0.197500 rpy=0.000000 0.000000 0.000000
- joint joint_3: origin xyz=0.000000 0.000000 0.445000 rpy=0.000000 1.919862175 0.000000 -> xyz=0.000000 0.000000 0.445000 rpy=0.000000 0.000000 0.000000

Commit message: Add default state

File: denso_robot_descriptions/vs087_description/vs087.urdf (robot description, URDF)
Before this commit: robot vs087, 8 links, 7 joints
Joints:
- joint joint_1: limit lower=-2.96706 upper=2.96706 effort=1 velocity=1 -> lower=-2.96706 upper=2.96706 effort=1 velocity=3.14159265358979
- joint joint_2: limit lower=-1.745329 upper=2.356194 effort=1 velocity=1 -> lower=-1.745329 upper=2.356194 effort=1 velocity=2.87979326579064
- joint joint_3: limit lower=-2.373648 upper=2.670354 effort=1 velocity=1 -> lower=-2.373648 upper=2.670354 effort=1 velocity=3.45575191894877
- joint joint_4: limit lower=-4.712389 upper=4.712389 effort=1 velocity=1 -> lower=-4.712389 upper=4.712389 effort=1 velocity=4.31968989868597
- joint joint_5: limit lower=-2.094395 upper=2.094395 effort=1 velocity=1 -> lower=-2.094395 upper=2.094395 effort=1 velocity=4.31968989868597
- joint joint_6: limit lower=-6.283185 upper=6.283185 effort=1 velocity=1 -> lower=-6.283185 upper=6.283185 effort=1 velocity=6.91150383789755
