Commit message: [modify] joint limit

File: denso_robot_descriptions/vs087_description/vs087_j3_pm5deg.urdf (robot description, URDF)
Before this commit: robot vs087, 8 links, 7 joints
Joints:
- joint joint_3: limit lower=-2.32129 upper=2.61799 effort=1 velocity=3.45575191894877 -> lower=-2.28638 upper=2.58309 effort=1 velocity=3.45575191894877

File: denso_robot_descriptions/vs087_description/vs087_original.urdf (robot description, URDF)
Before this commit: robot vs087, 8 links, 7 joints
Joints:
- joint joint_3: limit lower=-2.32129 upper=2.61799 effort=1 velocity=3.45575191894877 -> lower=-2.373648 upper=2.670354 effort=1 velocity=3.45575191894877
