Commit message: [fix] warnings

File: denso_robot_descriptions/vs087_description/vs087.urdf.xacro (robot description, xacro)
@@ -59,8 +59,8 @@
 		<type>transmission_interface/SimpleTransmission</type>
 		<joint name="joint_1">
-			<hardwareInterface>PositionJointInterface</hardwareInterface>
+			<hardwareInterface>hardware_interface/PositionJointInterface</hardwareInterface>
 		</joint>
 		<actuator name="motor_1">
-			<hardwareInterface>PositionJointInterface</hardwareInterface>
+			<hardwareInterface>hardware_interface/PositionJointInterface</hardwareInterface>
 			<mechanicalReduction>1</mechanicalReduction>
 		</actuator>
@@ -96,8 +96,8 @@
 		<type>transmission_interface/SimpleTransmission</type>
 		<joint name="joint_2">
-			<hardwareInterface>PositionJointInterface</hardwareInterface>
+			<hardwareInterface>hardware_interface/PositionJointInterface</hardwareInterface>
 		</joint>
 		<actuator name="motor_2">
-			<hardwareInterface>PositionJointInterface</hardwareInterface>
+			<hardwareInterface>hardware_interface/PositionJointInterface</hardwareInterface>
 			<mechanicalReduction>1</mechanicalReduction>
 		</actuator>
@@ -127,5 +127,5 @@
 		<origin rpy="0.000000 0.000000 0.000000" xyz="0.000000 0.000000 0.445000" />
 		<axis xyz="-0.000000 1.000000 -0.000000" />
-		<limit effort="1" lower="-2.373648" upper="2.670354" velocity="3.45575191894877" />
+		<limit effort="1" lower="-2.32129" upper="2.61799" velocity="3.45575191894877" />
 		<dynamics damping="0" friction="0" />
 	</joint>
@@ -133,8 +133,8 @@
 		<type>transmission_interface/SimpleTransmission</type>
 		<joint name="joint_3">
-			<hardwareInterface>PositionJointInterface</hardwareInterface>
+			<hardwareInterface>hardware_interface/PositionJointInterface</hardwareInterface>
 		</joint>
 		<actuator name="motor_3">
-			<hardwareInterface>PositionJointInterface</hardwareInterface>
+			<hardwareInterface>hardware_interface/PositionJointInterface</hardwareInterface>
 			<mechanicalReduction>1</mechanicalReduction>
 		</actuator>
@@ -170,8 +170,8 @@
 		<type>transmission_interface/SimpleTransmission</type>
 		<joint name="joint_4">
-			<hardwareInterface>PositionJointInterface</hardwareInterface>
+			<hardwareInterface>hardware_interface/PositionJointInterface</hardwareInterface>
 		</joint>
 		<actuator name="motor_4">
-			<hardwareInterface>PositionJointInterface</hardwareInterface>
+			<hardwareInterface>hardware_interface/PositionJointInterface</hardwareInterface>
 			<mechanicalReduction>1</mechanicalReduction>
 		</actuator>
@@ -207,8 +207,8 @@
 		<type>transmission_interface/SimpleTransmission</type>
 		<joint name="joint_5">
-			<hardwareInterface>PositionJointInterface</hardwareInterface>
+			<hardwareInterface>hardware_interface/PositionJointInterface</hardwareInterface>
 		</joint>
 		<actuator name="motor_5">
-			<hardwareInterface>PositionJointInterface</hardwareInterface>
+			<hardwareInterface>hardware_interface/PositionJointInterface</hardwareInterface>
 			<mechanicalReduction>1</mechanicalReduction>
 		</actuator>
@@ -244,8 +244,8 @@
 		<type>transmission_interface/SimpleTransmission</type>
 		<joint name="joint_6">
-			<hardwareInterface>PositionJointInterface</hardwareInterface>
+			<hardwareInterface>hardware_interface/PositionJointInterface</hardwareInterface>
 		</joint>
 		<actuator name="motor_6">
-			<hardwareInterface>PositionJointInterface</hardwareInterface>
+			<hardwareInterface>hardware_interface/PositionJointInterface</hardwareInterface>
 			<mechanicalReduction>1</mechanicalReduction>
 		</actuator>
