Commit message: [change] directory structure for vs060 description

File: denso_robot_descriptions/vs060_description/vs060/vs060.urdf (robot description, URDF)
Before this commit: robot vs060, 8 links, 7 joints
Links:
- link J1: geometry collision mesh filename=package://denso_robot_descriptions/vs060_description/vs060/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 scale=1 1 1; visual mesh filename=package://denso_robot_descriptions/vs060_description/vs060/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 scale=1 1 1
- link J2: geometry collision mesh filename=package://denso_robot_descriptions/vs060_description/vs060/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 scale=1 1 1; visual mesh filename=package://denso_robot_descriptions/vs060_description/vs060/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 scale=1 1 1
- link J3: geometry collision mesh filename=package://denso_robot_descriptions/vs060_description/vs060/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 scale=1 1 1; visual mesh filename=package://denso_robot_descriptions/vs060_description/vs060/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 scale=1 1 1
- link J4: geometry collision mesh filename=package://denso_robot_descriptions/vs060_description/vs060/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 scale=1 1 1; visual mesh filename=package://denso_robot_descriptions/vs060_description/vs060/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 scale=1 1 1
- link J5: geometry collision mesh filename=package://denso_robot_descriptions/vs060_description/vs060/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 scale=1 1 1; visual mesh filename=package://denso_robot_descriptions/vs060_description/vs060/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 scale=1 1 1
- link J6: geometry collision mesh filename=package://denso_robot_descriptions/vs060_description/vs060/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 scale=1 1 1; visual mesh filename=package://denso_robot_descriptions/vs060_description/vs060/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 scale=1 1 1
- link base_link: geometry collision mesh filename=package://denso_robot_descriptions/vs060_description/vs060/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 scale=1 1 1; visual mesh filename=package://denso_robot_descriptions/vs060_description/vs060/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 scale=1 1 1
