Commit message: [change] directory structure for vs087 description

File: denso_robot_descriptions/vs087_description/vs087/vs087.urdf (robot description, URDF)
Before this commit: robot vs087, 8 links, 7 joints
Links:
- link J1: geometry collision mesh filename=package://denso_robot_descriptions/vs087_description/vs087/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 scale=1 1 1; visual mesh filename=package://denso_robot_descriptions/vs087_description/vs087/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 scale=1 1 1
- link J2: geometry collision mesh filename=package://denso_robot_descriptions/vs087_description/vs087/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 scale=1 1 1; visual mesh filename=package://denso_robot_descriptions/vs087_description/vs087/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 scale=1 1 1
- link J3: geometry collision mesh filename=package://denso_robot_descriptions/vs087_description/vs087/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 scale=1 1 1; visual mesh filename=package://denso_robot_descriptions/vs087_description/vs087/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 scale=1 1 1
- link J4: geometry collision mesh filename=package://denso_robot_descriptions/vs087_description/vs087/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 scale=1 1 1; visual mesh filename=package://denso_robot_descriptions/vs087_description/vs087/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 scale=1 1 1
- link J5: geometry collision mesh filename=package://denso_robot_descriptions/vs087_description/vs087/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 scale=1 1 1; visual mesh filename=package://denso_robot_descriptions/vs087_description/vs087/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 scale=1 1 1
- link J6: geometry collision mesh filename=package://denso_robot_descriptions/vs087_description/vs087/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 scale=1 1 1; visual mesh filename=package://denso_robot_descriptions/vs087_description/vs087/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 scale=1 1 1
- link base_link: geometry collision mesh filename=package://denso_robot_descriptions/vs087_description/vs087/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 scale=1 1 1; visual mesh filename=package://denso_robot_descriptions/vs087_description/vs087/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 scale=1 1 1
Joints:
- joint joint_3: limit lower=-2.28638 upper=2.58309 effort=1 velocity=3.45575191894877 -> lower=-2.32129 upper=2.61799 effort=1 velocity=3.45575191894877

File: denso_robot_descriptions/vs087_description/vs087/vs087.urdf.xacro (robot description, xacro)
@@ -14,11 +14,11 @@
 			<origin rpy="0 0 0" xyz="0 0 0" />
 			<geometry>
-				<mesh filename="package://denso_robot_descriptions/vs087_description/base_link.dae" scale="1 1 1" />
-			</geometry>
-		</visual>
-		<collision>
-			<origin rpy="0 0 0" xyz="0 0 0" />
-			<geometry>
-				<mesh filename="package://denso_robot_descriptions/vs087_description/base_link.dae" scale="1 1 1" />
+				<mesh filename="package://denso_robot_descriptions/vs087_description/vs087/meshes/base_link.dae" scale="1 1 1" />
+			</geometry>
+		</visual>
+		<collision>
+			<origin rpy="0 0 0" xyz="0 0 0" />
+			<geometry>
+				<mesh filename="package://denso_robot_descriptions/vs087_description/vs087/meshes/base_link.dae" scale="1 1 1" />
 			</geometry>
 		</collision>
@@ -33,11 +33,11 @@
 			<origin rpy="0 0 0" xyz="0 0 0" />
 			<geometry>
-				<mesh filename="package://denso_robot_descriptions/vs087_description/J1.dae" scale="1 1 1" />
-			</geometry>
-		</visual>
-		<collision>
-			<origin rpy="0 0 0" xyz="0 0 0" />
-			<geometry>
-				<mesh filename="package://denso_robot_descriptions/vs087_description/J1.dae" scale="1 1 1" />
+				<mesh filename="package://denso_robot_descriptions/vs087_description/vs087/meshes/J1.dae" scale="1 1 1" />
+			</geometry>
+		</visual>
+		<collision>
+			<origin rpy="0 0 0" xyz="0 0 0" />
+			<geometry>
+				<mesh filename="package://denso_robot_descriptions/vs087_description/vs087/meshes/J1.dae" scale="1 1 1" />
 			</geometry>
 		</collision>
@@ -59,8 +59,8 @@
 		<type>transmission_interface/SimpleTransmission</type>
 		<joint name="joint_1">
-			<hardwareInterface>PositionJointInterface</hardwareInterface>
+			<hardwareInterface>hardware_interface/PositionJointInterface</hardwareInterface>
 		</joint>
 		<actuator name="motor_1">
-			<hardwareInterface>PositionJointInterface</hardwareInterface>
+			<hardwareInterface>hardware_interface/PositionJointInterface</hardwareInterface>
 			<mechanicalReduction>1</mechanicalReduction>
 		</actuator>
@@ -70,11 +70,11 @@
 			<origin rpy="0 0 0" xyz="0 0 0" />
 			<geometry>
-				<mesh filename="package://denso_robot_descriptions/vs087_description/J2.dae" scale="1 1 1" />
-			</geometry>
-		</visual>
-		<collision>
-			<origin rpy="0 0 0" xyz="0 0 0" />
-			<geometry>
-				<mesh filename="package://denso_robot_descriptions/vs087_description/J2.dae" scale="1 1 1" />
+				<mesh filename="package://denso_robot_descriptions/vs087_description/vs087/meshes/J2.dae" scale="1 1 1" />
+			</geometry>
+		</visual>
+		<collision>
+			<origin rpy="0 0 0" xyz="0 0 0" />
+			<geometry>
+				<mesh filename="package://denso_robot_descriptions/vs087_description/vs087/meshes/J2.dae" scale="1 1 1" />
 			</geometry>
 		</collision>
@@ -96,8 +96,8 @@
 		<type>transmission_interface/SimpleTransmission</type>
 		<joint name="joint_2">
-			<hardwareInterface>PositionJointInterface</hardwareInterface>
+			<hardwareInterface>hardware_interface/PositionJointInterface</hardwareInterface>
 		</joint>
 		<actuator name="motor_2">
-			<hardwareInterface>PositionJointInterface</hardwareInterface>
+			<hardwareInterface>hardware_interface/PositionJointInterface</hardwareInterface>
 			<mechanicalReduction>1</mechanicalReduction>
 		</actuator>
@@ -107,11 +107,11 @@
 			<origin rpy="0 0 0" xyz="0 0 0" />
 			<geometry>
-				<mesh filename="package://denso_robot_descriptions/vs087_description/J3.dae" scale="1 1 1" />
-			</geometry>
-		</visual>
-		<collision>
-			<origin rpy="0 0 0" xyz="0 0 0" />
-			<geometry>
-				<mesh filename="package://denso_robot_descriptions/vs087_description/J3.dae" scale="1 1 1" />
+				<mesh filename="package://denso_robot_descriptions/vs087_description/vs087/meshes/J3.dae" scale="1 1 1" />
+			</geometry>
+		</visual>
+		<collision>
+			<origin rpy="0 0 0" xyz="0 0 0" />
+			<geometry>
+				<mesh filename="package://denso_robot_descriptions/vs087_description/vs087/meshes/J3.dae" scale="1 1 1" />
 			</geometry>
 		</collision>
@@ -127,5 +127,5 @@
 		<origin rpy="0.000000 0.000000 0.000000" xyz="0.000000 0.000000 0.445000" />
 		<axis xyz="-0.000000 1.000000 -0.000000" />
-		<limit effort="1" lower="-2.373648" upper="2.670354" velocity="3.45575191894877" />
+		<limit effort="1" lower="-2.32129" upper="2.61799" velocity="3.45575191894877" />
 		<dynamics damping="0" friction="0" />
 	</joint>
@@ -133,8 +133,8 @@
 		<type>transmission_interface/SimpleTransmission</type>
 		<joint name="joint_3">
-			<hardwareInterface>PositionJointInterface</hardwareInterface>
+			<hardwareInterface>hardware_interface/PositionJointInterface</hardwareInterface>
 		</joint>
 		<actuator name="motor_3">
-			<hardwareInterface>PositionJointInterface</hardwareInterface>
+			<hardwareInterface>hardware_interface/PositionJointInterface</hardwareInterface>
 			<mechanicalReduction>1</mechanicalReduction>
 		</actuator>
@@ -144,11 +144,11 @@
 			<origin rpy="0 0 0" xyz="0 0 0" />
 			<geometry>
-				<mesh filename="package://denso_robot_descriptions/vs087_description/J4.dae" scale="1 1 1" />
-			</geometry>
-		</visual>
-		<collision>
-			<origin rpy="0 0 0" xyz="0 0 0" />
-			<geometry>
-				<mesh filename="package://denso_robot_descriptions/vs087_description/J4.dae" scale="1 1 1" />
+				<mesh filename="package://denso_robot_descriptions/vs087_description/vs087/meshes/J4.dae" scale="1 1 1" />
+			</geometry>
+		</visual>
+		<collision>
+			<origin rpy="0 0 0" xyz="0 0 0" />
+			<geometry>
+				<mesh filename="package://denso_robot_descriptions/vs087_description/vs087/meshes/J4.dae" scale="1 1 1" />
 			</geometry>
 		</collision>
@@ -170,8 +170,8 @@
 		<type>transmission_interface/SimpleTransmission</type>
 		<joint name="joint_4">
-			<hardwareInterface>PositionJointInterface</hardwareInterface>
+			<hardwareInterface>hardware_interface/PositionJointInterface</hardwareInterface>
 		</joint>
 		<actuator name="motor_4">
-			<hardwareInterface>PositionJointInterface</hardwareInterface>
+			<hardwareInterface>hardware_interface/PositionJointInterface</hardwareInterface>
 			<mechanicalReduction>1</mechanicalReduction>
 		</actuator>
@@ -181,11 +181,11 @@
 			<origin rpy="0 0 0" xyz="0 0 0" />
 			<geometry>
-				<mesh filename="package://denso_robot_descriptions/vs087_description/J5.dae" scale="1 1 1" />
-			</geometry>
-		</visual>
-		<collision>
-			<origin rpy="0 0 0" xyz="0 0 0" />
-			<geometry>
-				<mesh filename="package://denso_robot_descriptions/vs087_description/J5.dae" scale="1 1 1" />
+				<mesh filename="package://denso_robot_descriptions/vs087_description/vs087/meshes/J5.dae" scale="1 1 1" />
+			</geometry>
+		</visual>
+		<collision>
+			<origin rpy="0 0 0" xyz="0 0 0" />
+			<geometry>
+				<mesh filename="package://denso_robot_descriptions/vs087_description/vs087/meshes/J5.dae" scale="1 1 1" />
 			</geometry>
 		</collision>
@@ -207,8 +207,8 @@
 		<type>transmission_interface/SimpleTransmission</type>
 		<joint name="joint_5">
-			<hardwareInterface>PositionJointInterface</hardwareInterface>
+			<hardwareInterface>hardware_interface/PositionJointInterface</hardwareInterface>
 		</joint>
 		<actuator name="motor_5">
-			<hardwareInterface>PositionJointInterface</hardwareInterface>
+			<hardwareInterface>hardware_interface/PositionJointInterface</hardwareInterface>
 			<mechanicalReduction>1</mechanicalReduction>
 		</actuator>
@@ -218,11 +218,11 @@
 			<origin rpy="0 0 0" xyz="0 0 0" />
 			<geometry>
-				<mesh filename="package://denso_robot_descriptions/vs087_description/J6.dae" scale="1 1 1" />
-			</geometry>
-		</visual>
-		<collision>
-			<origin rpy="0 0 0" xyz="0 0 0" />
-			<geometry>
-				<mesh filename="package://denso_robot_descriptions/vs087_description/J6.dae" scale="1 1 1" />
+				<mesh filename="package://denso_robot_descriptions/vs087_description/vs087/meshes/J6.dae" scale="1 1 1" />
+			</geometry>
+		</visual>
+		<collision>
+			<origin rpy="0 0 0" xyz="0 0 0" />
+			<geometry>
+				<mesh filename="package://denso_robot_descriptions/vs087_description/vs087/meshes/J6.dae" scale="1 1 1" />
 			</geometry>
 		</collision>
@@ -244,8 +244,8 @@
 		<type>transmission_interface/SimpleTransmission</type>
 		<joint name="joint_6">
-			<hardwareInterface>PositionJointInterface</hardwareInterface>
+			<hardwareInterface>hardware_interface/PositionJointInterface</hardwareInterface>
 		</joint>
 		<actuator name="motor_6">
-			<hardwareInterface>PositionJointInterface</hardwareInterface>
+			<hardwareInterface>hardware_interface/PositionJointInterface</hardwareInterface>
 			<mechanicalReduction>1</mechanicalReduction>
 		</actuator>

File: denso_robot_descriptions/vs087_description/vs087/vs087_j3_pm5deg.urdf (robot description, URDF)
Before this commit: robot vs087, 8 links, 7 joints
Links:
- link J1: geometry collision mesh filename=package://denso_robot_descriptions/vs087_description/vs087/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 scale=1 1 1; visual mesh filename=package://denso_robot_descriptions/vs087_description/vs087/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 scale=1 1 1
- link J2: geometry collision mesh filename=package://denso_robot_descriptions/vs087_description/vs087/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 scale=1 1 1; visual mesh filename=package://denso_robot_descriptions/vs087_description/vs087/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 scale=1 1 1
- link J3: geometry collision mesh filename=package://denso_robot_descriptions/vs087_description/vs087/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 scale=1 1 1; visual mesh filename=package://denso_robot_descriptions/vs087_description/vs087/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 scale=1 1 1
- link J4: geometry collision mesh filename=package://denso_robot_descriptions/vs087_description/vs087/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 scale=1 1 1; visual mesh filename=package://denso_robot_descriptions/vs087_description/vs087/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 scale=1 1 1
- link J5: geometry collision mesh filename=package://denso_robot_descriptions/vs087_description/vs087/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 scale=1 1 1; visual mesh filename=package://denso_robot_descriptions/vs087_description/vs087/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 scale=1 1 1
- link J6: geometry collision mesh filename=package://denso_robot_descriptions/vs087_description/vs087/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 scale=1 1 1; visual mesh filename=package://denso_robot_descriptions/vs087_description/vs087/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 scale=1 1 1
- link base_link: geometry collision mesh filename=package://denso_robot_descriptions/vs087_description/vs087/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 scale=1 1 1; visual mesh filename=package://denso_robot_descriptions/vs087_description/vs087/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 scale=1 1 1
Joints:
- joint joint_3: limit lower=-2.32129 upper=2.61799 effort=1 velocity=3.45575191894877 -> lower=-2.28638 upper=2.58309 effort=1 velocity=3.45575191894877

File: denso_robot_descriptions/vs087_description/vs087/vs087_original.urdf (robot description, URDF)
Before this commit: robot vs087, 8 links, 7 joints
Links:
- link J1: geometry collision mesh filename=package://denso_robot_descriptions/vs087_description/vs087/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 scale=1 1 1; visual mesh filename=package://denso_robot_descriptions/vs087_description/vs087/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 scale=1 1 1
- link J2: geometry collision mesh filename=package://denso_robot_descriptions/vs087_description/vs087/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 scale=1 1 1; visual mesh filename=package://denso_robot_descriptions/vs087_description/vs087/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 scale=1 1 1
- link J3: geometry collision mesh filename=package://denso_robot_descriptions/vs087_description/vs087/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 scale=1 1 1; visual mesh filename=package://denso_robot_descriptions/vs087_description/vs087/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 scale=1 1 1
- link J4: geometry collision mesh filename=package://denso_robot_descriptions/vs087_description/vs087/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 scale=1 1 1; visual mesh filename=package://denso_robot_descriptions/vs087_description/vs087/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 scale=1 1 1
- link J5: geometry collision mesh filename=package://denso_robot_descriptions/vs087_description/vs087/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 scale=1 1 1; visual mesh filename=package://denso_robot_descriptions/vs087_description/vs087/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 scale=1 1 1
- link J6: geometry collision mesh filename=package://denso_robot_descriptions/vs087_description/vs087/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 scale=1 1 1; visual mesh filename=package://denso_robot_descriptions/vs087_description/vs087/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 scale=1 1 1
- link base_link: geometry collision mesh filename=package://denso_robot_descriptions/vs087_description/vs087/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 scale=1 1 1; visual mesh filename=package://denso_robot_descriptions/vs087_description/vs087/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 scale=1 1 1
Joints:
- joint joint_3: limit lower=-2.32129 upper=2.61799 effort=1 velocity=3.45575191894877 -> lower=-2.373648 upper=2.670354 effort=1 velocity=3.45575191894877

File: denso_robot_descriptions/vs087_description/vs087_with_2_kinects/vs087_with_2_kinects.urdf.xacro (robot description, xacro)
@@ -4,5 +4,5 @@
   <xacro:include filename="$(find kinect_bringup)/urdf/sensor/kinect.urdf.xacro"/>
   <xacro:include filename="$(find kinect_bringup)/urdf/sensor/kinect.gazebo.xacro"/>
-  <xacro:include filename="$(find denso_robot_descriptions)/vs087_description/vs087.urdf.xacro"/>
+  <xacro:include filename="$(find denso_robot_descriptions)/vs087_description/vs087/vs087.urdf.xacro"/>
   <!-- add Kinect V2 -->
   <!-- kinect_center -->
