Commit message: Modify joint limit

File: denso_robot_descriptions/vs087_description/vs087/vs087.urdf.xacro (robot description, xacro)
@@ -238,5 +238,6 @@
 		<origin rpy="0.000000 0.000000 0.000000" xyz="0.000000 0.000000 0.080000" />
 		<axis xyz="-0.000000 -0.000000 1.000000" />
-		<limit effort="1" lower="2.13750473492" upper="6.283185" velocity="6.91150383789755" />
+		<!-- <limit effort="1" lower="2.13750473492" upper="6.283185" velocity="6.91150383789755" /> -->
+		<limit effort="1" lower="0.0" upper="6.283185" velocity="6.91150383789755" />
 		<dynamics damping="0" friction="0" />
 	</joint>

File: denso_robot_descriptions/vs087_description/vs087_and_mhand_with_3_kinects/vs087_and_mhand_with_3_kinects.urdf.xacro (robot description, xacro)
@@ -1,6 +1,6 @@
 <?xml version="1.0"?>
 <robot name="vs087" xmlns:xacro="http://ros.org/wiki/xacro">
-  <!-- <xacro:include filename="$(find denso_robot_descriptions)/vs087_description/vs087/vs087.urdf.xacro"/> -->
-  <xacro:include filename="$(find denso_robot_descriptions)/vs087_description/vs087_and_mhand/vs087_limited_joints_for_mhand.urdf.xacro"/>
+  <xacro:include filename="$(find denso_robot_descriptions)/vs087_description/vs087/vs087.urdf.xacro"/>
+  <!-- <xacro:include filename="$(find denso_robot_descriptions)/vs087_description/vs087_and_mhand/vs087_limited_joints_for_mhand.urdf.xacro"/> -->
   <xacro:include filename="$(find mhand_description)/robots/mhand.urdf.xacro"/>
   <xacro:include filename="$(find kinect_bringup)/urdf/sensor/kinect.urdf.xacro"/>
