Commit message: [modify] coordinate

File: denso_robot_descriptions/vs087_description/vs087_and_mhand/vs087_and_mhand.urdf.xacro (robot description, xacro)
@@ -4,5 +4,5 @@
   <xacro:include filename="$(find mhand_description)/robots/mhand.urdf.xacro"/>
   <joint name="gripper_joint" type="fixed">
-  <origin xyz="0 0 0" rpy="0 ${pi} ${pi}"/>
+    <origin xyz="0 0 0" rpy="0 0 0"/>
   <parent link="J6"/>
   <child link="hand_link"/>
