Commit message: [modify] calibrated kinect_center

File: denso_robot_descriptions/vs087_description/vs087_and_mhand_with_3_kinects/vs087_and_mhand_with_3_kinects.urdf.xacro (robot description, xacro)
@@ -18,5 +18,5 @@
   <!-- Joint -->
   <joint name="joint_kinect_center" type="fixed">
-    <origin xyz="1.265 0.04 0.515" rpy="0 0.3780 -3.123" />
+    <origin xyz="1.2297 0.1072 0.4985" rpy="-0.0047 0.5886 3.098" />>
     <parent link="world"/>
     <child link="kinect_center_link"/>

Commit message: [modified] calibrated kinect_center position

File: denso_robot_descriptions/vs087_description/vs087_and_mhand_with_3_kinects/vs087_and_mhand_with_3_kinects.urdf.xacro (robot description, xacro)
@@ -18,5 +18,6 @@
   <!-- Joint -->
   <joint name="joint_kinect_center" type="fixed">
-    <origin xyz="1.2297 0.1072 0.4985" rpy="-0.0047 0.5886 3.098" />>
+    <!-- <origin xyz="1.2297 0.1072 0.4985" rpy="-0.0047 0.5886 3.098" />> -->
+    <origin xyz="1.2346 0.055 0.7236" rpy="-0.0184 0.5637 3.046" />
     <parent link="world"/>
     <child link="kinect_center_link"/>

Commit message: [modified] calibrated kinect_center

File: denso_robot_descriptions/vs087_description/vs087_and_mhand_with_3_kinects/vs087_and_mhand_with_3_kinects.urdf.xacro (robot description, xacro)
@@ -19,5 +19,5 @@
   <joint name="joint_kinect_center" type="fixed">
     <!-- <origin xyz="1.2297 0.1072 0.4985" rpy="-0.0047 0.5886 3.098" />> -->
-    <origin xyz="1.2346 0.055 0.7236" rpy="-0.0184 0.5637 3.046" />
+    <origin xyz="0.8567 0.0762 0.9535" rpy="-0.0338 0.8795 3.0507" />
     <parent link="world"/>
     <child link="kinect_center_link"/>
