Commit message: [modified] to connect real robot with robotiq hand

File: denso_robot_descriptions/vs087_description/vs087_and_robotiq/vs087_and_robotiq.urdf.xacro (robot description, xacro)
@@ -242,5 +242,5 @@
   <joint name="gripper_joint" type="fixed">
     <!-- <origin xyz="0 0 0.038" rpy="${pi/2} 0 ${pi}"/> -->
-    <origin xyz="0 0 0.038" rpy="${pi/2} 0 0"/>
+    <origin xyz="0 0 0.038" rpy="${pi/2} 0 ${-pi/6}"/>
   <parent link="J6"/>
   <child link="palm"/>
