Commit message: [modify] kinect position and fix move_group for real robot

File: denso_robot_descriptions/vs087_description/vs087_and_robotiq_with_1_kinect/vs087_and_robotiq_with_1_kinect.urdf.xacro (robot description, xacro)
@@ -13,5 +13,6 @@
   <joint name="joint_kinect_center" type="fixed">
     <!-- <origin xyz="1.2297 0.1072 0.4985" rpy="-0.0047 0.5886 3.098" />> -->
-    <origin xyz="0.8567 0.0762 0.9535" rpy="-0.0338 0.8795 3.0507" />
+    <!-- <origin xyz="0.8567 0.0762 0.9535" rpy="-0.0338 0.8795 3.0507" /> -->
+    <origin xyz="0.8834 0.0504 0.9911" rpy="-0.0078 0.6452 -3.1362" />
     <parent link="world"/>
     <child link="kinect_center_link"/>
