Commit message: Add hardware interface

File: denso_robot_description/urdf/common.xacro (robot description, xacro)
@@ -7,12 +7,12 @@
         rpy="0 0 0" />
       <mass
-        value="0.01" />
+        value="1" />
       <inertia
-        ixx="0.001"
+        ixx="1"
         ixy="0.0"
         ixz="0.0"
-        iyy="0.001"
+        iyy="1"
         iyz="0.0"
-        izz="0.001" />
+        izz="1" />
     </inertial>
   </xacro:macro>

File: denso_robot_description/urdf/denso_robot.urdf.xacro (robot description, xacro)
@@ -3,10 +3,14 @@
   <!-- Use this if parameters are set from the launch file, otherwise delete -->
   <xacro:arg name="prefix" default="" />
-  <xacro:arg name="use_mock_hardware" default="false" />
-  <xacro:arg name="mock_sensor_commands" default="false" />
   <xacro:arg name="sim_gazebo_classic" default="false" />
   <xacro:arg name="sim_gazebo" default="false" />
   <xacro:arg name="simulation_controllers" default="" />
+  <xacro:arg name="robot_ip" default="192.168.0.1" />
+  <xacro:arg name="robot_port" default="5900"/>
+  <xacro:arg name="send_format" default="288"/>
+  <xacro:arg name="recv_format" default="292"/>
+  <!-- Import Denso Robot Model -->
   <xacro:include filename="$(find denso_robot_description)/urdf/denso_robot/denso_robot_macro.xacro"/>
+  <!-- Import ROS2 Control -->
   <xacro:include filename="$(find denso_robot_description)/urdf/denso_robot/denso_robot_macro.ros2_control.xacro"/>
   <!-- create link fixed to the "world" -->
@@ -17,21 +21,11 @@
     <origin xyz="0 0 0" rpy="0 0 0" />          <!-- position robot in the world -->
   </xacro:denso_robot>
-  <xacro:denso_robot_ros2_control
-    name="denso_robot"
+  <xacro:denso_robot_ros2_control name="$(arg prefix)denso_control"
     prefix="$(arg prefix)"
-    use_mock_hardware="$(arg use_mock_hardware)"
-    mock_sensor_commands="$(arg mock_sensor_commands)"
-    sim_gazebo_classic="$(arg sim_gazebo_classic)"
-    sim_gazebo="$(arg sim_gazebo)"/>
-  <xacro:if value="$(arg sim_gazebo_classic)">
-    <!-- Gazebo plugins -->
-    <gazebo reference="world">
-    </gazebo>
-    <gazebo>
-      <plugin filename="libgazebo_ros2_control.so" name="gazebo_ros2_control">
-        <parameters>$(arg simulation_controllers)</parameters>
-      </plugin>
-    </gazebo>
-  </xacro:if>
+    sim_gazebo="$(arg sim_gazebo)"
+    robot_ip="$(arg robot_ip)"
+    robot_port="$(arg robot_port)"
+    send_format="$(arg send_format)"
+    recv_format="$(arg recv_format)" />
   <xacro:if value="$(arg sim_gazebo)">
     <!-- Gazebo plugins -->

File: denso_robot_description/urdf/denso_robot/denso_robot_macro.ros2_control.xacro (robot description, xacro)
@@ -1,18 +1,14 @@
 <?xml version="1.0" encoding="UTF-8"?>
-<robot xmlns:xacro="http://wiki.ros.org/xacro">
-  <xacro:macro name="denso_robot_ros2_control" params="
-               name
-               prefix
-               use_mock_hardware:=^|false
-               mock_sensor_commands:=^|false
-               sim_gazebo_classic:=^|false
-               sim_gazebo:=^|false"
-               >
+<robot xmlns:xacro="http://www.ros.org/wiki/xacro">
+  <xacro:macro name="denso_robot_ros2_control" params="name prefix
+    sim_gazebo_classic:=^|false
+    sim_gazebo:=^|false
+    robot_ip:=^|192.168.0.1
+    robot_port:=^|5007
+    send_format
+    recv_format
+    controller_type:=^|8">
     <ros2_control name="${name}" type="system">
       <hardware>
-        <xacro:if value="${use_mock_hardware}">
-          <plugin>mock_components/GenericSystem</plugin>
-          <param name="mock_sensor_commands">${mock_sensor_commands}</param>
-        </xacro:if>
         <xacro:if value="${sim_gazebo_classic}">
           <plugin>gazebo_ros2_control/GazeboSystem</plugin>
@@ -21,95 +17,77 @@
           <plugin>ign_ros2_control/IgnitionSystem</plugin>
         </xacro:if>
-        <xacro:unless value="${use_mock_hardware or sim_gazebo_classic or sim_gazebo}">
-          <plugin>robot_hardware_inteface/RobotHardwareInteface</plugin>
+        <xacro:unless value="${sim_gazebo_classic or sim_gazebo}">
+          <plugin>denso_hw/denso_hw</plugin>
+          <param name="robot_ip">${robot_ip}</param>
+          <param name="robot_port">${robot_port}</param>
+          <param name="send_format">${send_format}</param>
+          <param name="recv_format">${recv_format}</param>
+          <param name="controller_type">${controller_type}</param>
         </xacro:unless>
       </hardware>
       <joint name="${prefix}joint1">
-        <command_interface name="position">     <!-- Add/Remove interfaces as needed -->
-          <param name="min">-1</param>
-          <param name="max">1</param>
+        <command_interface name="position">
+          <param name="min">${radians(-170)}</param>
+          <param name="max">${radians(170)}</param>
         </command_interface>
-        <state_interface name="position">
-          <param name="initial_value">0.0</param>
-        <state_interface/>
+        <state_interface name="position"/>
         <state_interface name="velocity"/>
-        <state_interface name="acceleration"/>
+        <state_interface name="effort"/>
       </joint>
       <joint name="${prefix}joint2">
-        <command_interface name="position">     <!-- Add/Remove interfaces as needed -->
-          <param name="min">-1</param>
-          <param name="max">1</param>
+        <command_interface name="position">
+          <param name="min">${radians(-100)}</param>
+          <param name="max">${radians(135)}</param>
         </command_interface>
-        <state_interface name="position">
-          <param name="initial_value">0.0</param>
-        <state_interface/>
+        <state_interface name="position"/>
         <state_interface name="velocity"/>
-        <state_interface name="acceleration"/>
+        <state_interface name="effort"/>
       </joint>
       <joint name="${prefix}joint3">
-        <command_interface name="position">     <!-- Add/Remove interfaces as needed -->
-          <param name="min">-1</param>
-          <param name="max">1</param>
+        <command_interface name="position">
+          <param name="min">${radians(-136)}</param>
+          <param name="max">${radians(153)}</param>
         </command_interface>
-        <state_interface name="position">
-          <param name="initial_value">0.0</param>
-        <state_interface/>
+        <state_interface name="position"/>
         <state_interface name="velocity"/>
-        <state_interface name="acceleration"/>
+        <state_interface name="effort"/>
       </joint>
       <joint name="${prefix}joint4">
-        <command_interface name="position">     <!-- Add/Remove interfaces as needed -->
-          <param name="min">-1</param>
-          <param name="max">1</param>
+        <command_interface name="position">
+          <param name="min">${radians(-270)}</param>
+          <param name="max">${radians(270)}</param>
         </command_interface>
-        <state_interface name="position">
-          <param name="initial_value">0.0</param>
-        <state_interface/>
+        <state_interface name="position"/>
         <state_interface name="velocity"/>
-        <state_interface name="acceleration"/>
+        <state_interface name="effort"/>
       </joint>
       <joint name="${prefix}joint5">
-        <command_interface name="position">     <!-- Add/Remove interfaces as needed -->
-          <param name="min">-1</param>
-          <param name="max">1</param>
+        <command_interface name="position">
+          <param name="min">${radians(-120)}</param>
+          <param name="max">${radians(120)}</param>
         </command_interface>
-        <state_interface name="position">
-          <param name="initial_value">0.0</param>
-        <state_interface/>
+        <state_interface name="position"/>
         <state_interface name="velocity"/>
-        <state_interface name="acceleration"/>
+        <state_interface name="effort"/>
       </joint>
       <joint name="${prefix}joint6">
-        <command_interface name="position">     <!-- Add/Remove interfaces as needed -->
-          <param name="min">-1</param>
-          <param name="max">1</param>
+        <command_interface name="position">
+          <param name="min">${radians(-360)}</param>
+          <param name="max">${radians(360)}</param>
         </command_interface>
-        <state_interface name="position">
-          <param name="initial_value">0.0</param>
-        <state_interface/>
+        <state_interface name="position"/>
         <state_interface name="velocity"/>
-        <state_interface name="acceleration"/>
+        <state_interface name="effort"/>
       </joint>
-      <sensor name="tcp_fts_sensor">            <!-- Remove/change sensors as needed -->
-        <state_interface name="fx"/>
-        <state_interface name="fy"/>
-        <state_interface name="fz"/>
-        <state_interface name="tx"/>
-        <state_interface name="ty"/>
-        <state_interface name="tz"/>
-        <param name="frame_id">tool0</param>    <!-- Change sensors as needed -->
-        <param name="min_fx">-100</param>
-        <param name="max_fx">100</param>
-        <param name="min_fy">-100</param>
-        <param name="max_fy">100</param>
-        <param name="min_fz">-200</param>
-        <param name="max_fz">200</param>
-        <param name="min_tx">-10</param>
-        <param name="max_tx">10</param>
-        <param name="min_ty">-10</param>
-        <param name="max_ty">10</param>
-        <param name="min_tz">-15</param>
-        <param name="max_tz">15</param>
-      </sensor>
+      <!-- Transmission -->
+      <transmission name="transmission">
+        <plugin>transmission_interface/SimpleTransmission</plugin>
+        <joint name="joint1" role="revolute"/>
+        <joint name="joint2" role="revolute"/>
+        <joint name="joint3" role="revolute"/>
+        <joint name="joint4" role="revolute"/>
+        <joint name="joint5" role="revolute"/>
+        <joint name="joint6" role="revolute"/>
+      </transmission>
     </ros2_control>
   </xacro:macro>

File: denso_robot_description/urdf/denso_robot/denso_robot_macro.xacro (robot description, xacro)
@@ -12,6 +12,5 @@
         <origin rpy="0 0 0" xyz="0 0 0" />
         <geometry>
-          <cylinder length="0.3" radius="0.3" />
-<!--           <mesh filename="package://denso_robot_description/meshes/denso_robot/visual/base_link.dae" /> -->
+          <mesh filename="package://denso_robot_description/meshes/denso_robot/visual/base_link.dae" />
         </geometry>
       </visual>
@@ -19,6 +18,5 @@
         <origin rpy="0 0 0" xyz="0 0 0" />
         <geometry>
-          <cylinder length="0.3" radius="0.3" />
-<!--           <mesh filename="package://denso_robot_description/meshes/denso_robot/collision/base_link.stl" /> -->
+          <mesh filename="package://denso_robot_description/meshes/denso_robot/visual/base_link.dae" />
         </geometry>
       </collision>
@@ -32,6 +30,5 @@
         <origin xyz="0 0 0" rpy="0 0 0" />
         <geometry>
-          <cylinder length="0.3" radius="0.15" />
-<!--           <mesh filename="package://denso_robot_description/meshes/denso_robot/visual/link1.dae" /> -->
+          <mesh filename="package://denso_robot_description/meshes/denso_robot/visual/J1.dae" />
         </geometry>
       </visual>
@@ -39,6 +36,5 @@
         <origin xyz="0 0 0" rpy="0 0 0" />
         <geometry>
-          <cylinder length="0.3" radius="0.15" />
-<!--           <mesh filename="package://denso_robot_description/meshes/denso_robot/collision/link1.stl" /> -->
+          <mesh filename="package://denso_robot_description/meshes/denso_robot/visual/J1.dae" />
         </geometry>
       </collision>
@@ -52,6 +48,5 @@
         <origin xyz="0 0 0" rpy="0 0 0" />
         <geometry>
-          <cylinder length="0.8" radius="0.15" />
-<!--           <mesh filename="package://denso_robot_description/meshes/denso_robot/visual/link2.dae" /> -->
+          <mesh filename="package://denso_robot_description/meshes/denso_robot/visual/J2.dae" />
         </geometry>
       </visual>
@@ -59,6 +54,5 @@
         <origin xyz="0 0 0" rpy="0 0 0" />
         <geometry>
-          <cylinder length="0.8" radius="0.15" />
-<!--           <mesh filename="package://denso_robot_description/meshes/denso_robot/collision/link2.stl"  /> -->
+          <mesh filename="package://denso_robot_description/meshes/denso_robot/visual/J2.dae"  />
         </geometry>
       </collision>
@@ -72,6 +66,5 @@
         <origin xyz="0 0 0" rpy="0 0 0" />
         <geometry>
-          <cylinder length="0.5" radius="0.10" />
-<!--           <mesh filename="package://denso_robot_description/meshes/denso_robot/visual/link3.dae" /> -->
+          <mesh filename="package://denso_robot_description/meshes/denso_robot/visual/J3.dae" />
         </geometry>
       </visual>
@@ -79,6 +72,5 @@
         <origin xyz="0 0 0" rpy="0 0 0" />
         <geometry>
-          <cylinder length="0.5" radius="0.10" />
-<!--           <mesh filename="package://denso_robot_description/meshes/denso_robot/collision/link3.stl"  /> -->
+          <mesh filename="package://denso_robot_description/meshes/denso_robot/visual/J3.dae"  />
         </geometry>
       </collision>
@@ -92,6 +84,5 @@
         <origin xyz="0 0 0" rpy="0 0 0" />
         <geometry>
-          <cylinder length="0.1" radius="0.2" />
-<!--           <mesh filename="package://denso_robot_description/meshes/denso_robot/visual/link4.dae" /> -->
+          <mesh filename="package://denso_robot_description/meshes/denso_robot/visual/J4.dae" />
         </geometry>
       </visual>
@@ -99,6 +90,5 @@
         <origin xyz="0 0 0" rpy="0 0 0" />
         <geometry>
-          <cylinder length="0.1" radius="0.2" />
-<!--           <mesh filename="package://denso_robot_description/meshes/denso_robot/collision/link4.stl"  /> -->
+          <mesh filename="package://denso_robot_description/meshes/denso_robot/visual/J4.dae"  />
         </geometry>
       </collision>
@@ -112,6 +102,5 @@
         <origin xyz="0 0 0" rpy="0 0 0" />
         <geometry>
-          <cylinder length="0.2" radius="0.1" />
-<!--           <mesh filename="package://denso_robot_description/meshes/denso_robot/visual/link5.dae" /> -->
+          <mesh filename="package://denso_robot_description/meshes/denso_robot/visual/J5.dae" />
         </geometry>
       </visual>
@@ -119,6 +108,5 @@
         <origin xyz="0 0 0" rpy="0 0 0" />
         <geometry>
-          <cylinder length="0.2" radius="0.1" />
-<!--           <mesh filename="package://denso_robot_description/meshes/denso_robot/collision/link5.stl" /> -->
+          <mesh filename="package://denso_robot_description/meshes/denso_robot/visual/J5.dae" />
         </geometry>
       </collision>
@@ -132,6 +120,5 @@
         <origin xyz="0 0 0" rpy="0 0 0" />
         <geometry>
-          <cylinder length="0.05" radius="0.1" />
-<!--           <mesh filename="package://denso_robot_description/meshes/denso_robot/visual/link6.dae" /> -->
+          <mesh filename="package://denso_robot_description/meshes/denso_robot/visual/J6.dae" />
         </geometry>
       </visual>
@@ -139,6 +126,5 @@
         <origin xyz="0 0 0" rpy="0 0 0" />
         <geometry>
-          <cylinder length="0.05" radius="0.1" />
-<!--           <mesh filename="package://denso_robot_description/meshes/denso_robot/collision/link6.stl" /> -->
+          <mesh filename="package://denso_robot_description/meshes/denso_robot/visual/J6.dae" />
         </geometry>
       </collision>
@@ -147,12 +133,4 @@
     <link name="${prefix}tool0" />
     <!-- tool link -->
-<!-- START Delete if not needed -->
-    <!-- Standard frames for industrial robots. Also useful for manipulators.
-         (ROS-I specs - https://wiki.ros.org/Industrial/Tutorials/WorkingWithRosIndustrialRobotSupportPackages#Standardised_links_.2F_frames)-->
-    <!-- This frame should correspond to the BASE coordinate system of robot's controller.) -->
-    <link name="${prefix}base" />
-    <!-- Frame for mounting EEF models to a manipulator. x+ axis points forward (REP 103). -->
-    <link name="${prefix}flange" />
-<!-- END Delete if not needed  -->
     <!-- END LINKS -->
     <!-- JOINTS -->
@@ -165,49 +143,49 @@
     <!-- joint 1 -->
     <joint name="${prefix}joint1" type="revolute">
-      <origin xyz="0 0 0.3" rpy="${pi} 0 0" />
+      <origin xyz="0 0 0.197500" rpy="0 0 0" />
       <parent link="${prefix}base_link" />
       <child link="${prefix}link1" />
       <axis xyz="0 0 1" />
-      <limit effort="0" lower="${radians(-180)}" upper="${radians(180)}" velocity="${radians(180)}" />
+      <limit effort="0" lower="${radians(-170)}" upper="${radians(170)}" velocity="${radians(360)}" />
     </joint>
     <!-- joint 2 -->
     <joint name="${prefix}joint2" type="revolute">
-      <origin xyz="0 0 0.3" rpy="${pi/2} 0 0" />
+      <origin xyz="0.03 0 0.1975" rpy="0 0 0" />
       <parent link="${prefix}link1" />
       <child link="${prefix}link2" />
-      <axis xyz="0 0 1" />
-      <limit effort="0" lower="${radians(-180)}" upper="${radians(180)}" velocity="${radians(180)}" />
+      <axis xyz="0 1 0" />
+      <limit effort="0" lower="${radians(-100)}" upper="${radians(135)}" velocity="${radians(300)}" />
     </joint>
     <!-- joint 3 -->
     <joint name="${prefix}joint3" type="revolute">
-      <origin xyz="0.8 0 0" rpy="0 0 0" />
+      <origin xyz="0 0 0.445" rpy="0 0 0" />
       <parent link="${prefix}link2" />
       <child link="${prefix}link3" />
-      <axis xyz="0 0 1" />
-      <limit effort="0" lower="${radians(-90)}" upper="${radians(180)}" velocity="${radians(270)}" />
+      <axis xyz="0 1 0" />
+      <limit effort="0" lower="${radians(-136)}" upper="${radians(153)}" velocity="${radians(408)}" />
     </joint>
     <!-- joint 4 -->
     <joint name="${prefix}joint4" type="revolute">
-      <origin xyz="0 0.1 0" rpy="0 ${-pi/2} 0" />
+      <origin xyz="-0.02 0 0.287" rpy="0 0 0" />
       <parent link="${prefix}link3" />
       <child link="${prefix}link4" />
       <axis xyz="0 0 1" />
-      <limit effort="0" lower="${radians(-360)}" upper="${radians(360)}" velocity="${radians(360)}" />
+      <limit effort="0" lower="${radians(-270)}" upper="${radians(270)}" velocity="${radians(540)}" />
     </joint>
     <!-- joint 5 -->
     <joint name="${prefix}joint5" type="revolute">
-      <origin xyz="0 0 -0.1" rpy="0 ${pi/2} 0" />
+      <origin xyz="0 0 0.143" rpy="0 0 0" />
       <parent link="${prefix}link4" />
       <child link="${prefix}link5" />
-      <axis xyz="0 0 1" />
+      <axis xyz="0 1 0" />
       <limit effort="0" lower="${radians(-120)}" upper="${radians(120)}" velocity="${radians(540)}" />
     </joint>
     <!-- joint 6 -->
     <joint name="${prefix}joint6" type="revolute">
-      <origin xyz="0 0 0.1" rpy="0 ${-pi/2} 0" />
+      <origin xyz="0 0 0.08" rpy="0 0 0" />
       <parent link="${prefix}link5" />
       <child link="${prefix}link6" />
       <axis xyz="0 0 1" />
-      <limit effort="0" lower="${radians(-360)}" upper="${radians(360)}" velocity="${radians(720)}" />
+      <limit effort="0" lower="${radians(-360)}" upper="${radians(360)}" velocity="${radians(864)}" />
     </joint>
     <!-- tool frame - fixed frame -->
@@ -218,18 +196,4 @@
     </joint>
     <!-- END JOINTS -->
-<!-- START Delete if not needed -->
-    <!-- Standard frames for industrial robots. Also useful for manipulators.
-         (ROS-I specs - https://wiki.ros.org/Industrial/Tutorials/WorkingWithRosIndustrialRobotSupportPackages#Standardised_links_.2F_frames)-->
-    <joint name="${prefix}base_link-base_joint" type="fixed">
-      <origin xyz="0 0 0" rpy="0 0 0" />
-      <parent link="${prefix}base_link" />
-      <child link="${prefix}base" />
-    </joint>
-    <joint name="${prefix}tool0-flange_joint" type="fixed">
-      <origin xyz="0 0 0" rpy="0 0 0" />
-      <parent link="${prefix}tool0" />
-      <child link="${prefix}flange" />
-    </joint>
-<!-- END Delete if not needed  -->
   </xacro:macro>
 </robot>
