Commit message: Add Gazebo

File: denso_robot_description/urdf/denso_robot.urdf.xacro (robot description, xacro)
@@ -4,5 +4,5 @@
   <xacro:arg name="prefix" default="" />
   <xacro:arg name="sim_gazebo_classic" default="false" />
-  <xacro:arg name="sim_gazebo" default="false" />
+  <xacro:arg name="sim_gazebo" default="true" />
   <xacro:arg name="simulation_controllers" default="" />
   <xacro:arg name="robot_ip" default="192.168.0.1" />
@@ -31,11 +31,8 @@
     config_file="$(arg config_file)"/>
   <xacro:if value="$(arg sim_gazebo)">
-    <!-- Gazebo plugins -->
-    <gazebo reference="world">
-    </gazebo>
     <gazebo>
-      <plugin filename="libign_ros2_control-system.so" name="ign_ros2_control::IgnitionROS2ControlPlugin">
-        <parameters>$(arg simulation_controllers)</parameters>
-        <controller_manager_node_name>$(arg prefix)controller_manager</controller_manager_node_name>
+      <!-- Joint state publisher -->
+      <plugin filename="gz_ros2_control-system" name="gz_ros2_control::GazeboSimROS2ControlPlugin">
+        <parameters>$(find denso_robot_bringup)/config/denso_robot_gazebo_controllers.yaml</parameters>
       </plugin>
     </gazebo>

File: denso_robot_description/urdf/denso_robot/denso_robot_macro.ros2_control.xacro (robot description, xacro)
@@ -3,5 +3,5 @@
   <xacro:macro name="denso_robot_ros2_control" params="name prefix
     sim_gazebo_classic:=^|false
-    sim_gazebo:=^|false
+    sim_gazebo:=^|true
     robot_ip:=^|192.168.0.1
     robot_port:=^|5007
@@ -16,5 +16,5 @@
         </xacro:if>
         <xacro:if value="${sim_gazebo}">
-          <plugin>ign_ros2_control/IgnitionSystem</plugin>
+          <plugin>gz_ros2_control/GazeboSimSystem</plugin>
         </xacro:if>
         <xacro:unless value="${sim_gazebo_classic or sim_gazebo}">

File: denso_robot_description/urdf/denso_robot/denso_robot_macro.xacro (robot description, xacro)
@@ -147,5 +147,6 @@
       <child link="${prefix}link1" />
       <axis xyz="0 0 1" />
-      <limit effort="0" lower="${radians(-170)}" upper="${radians(170)}" velocity="${radians(360)}" />
+      <limit effort="1000" lower="${radians(-170)}" upper="${radians(170)}" velocity="${radians(360)}" />
+      <dynamics damping="0.7" friction="0.0"/>
     </joint>
     <!-- joint 2 -->
@@ -155,5 +156,6 @@
       <child link="${prefix}link2" />
       <axis xyz="0 1 0" />
-      <limit effort="0" lower="${radians(-100)}" upper="${radians(135)}" velocity="${radians(300)}" />
+      <limit effort="1000" lower="${radians(-100)}" upper="${radians(135)}" velocity="${radians(300)}" />
+      <dynamics damping="0.7" friction="0.0"/>
     </joint>
     <!-- joint 3 -->
@@ -163,5 +165,6 @@
       <child link="${prefix}link3" />
       <axis xyz="0 1 0" />
-      <limit effort="0" lower="${radians(-136)}" upper="${radians(153)}" velocity="${radians(408)}" />
+      <limit effort="1000" lower="${radians(-136)}" upper="${radians(153)}" velocity="${radians(408)}" />
+      <dynamics damping="0.7" friction="0.0"/>
     </joint>
     <!-- joint 4 -->
@@ -171,5 +174,6 @@
       <child link="${prefix}link4" />
       <axis xyz="0 0 1" />
-      <limit effort="0" lower="${radians(-270)}" upper="${radians(270)}" velocity="${radians(540)}" />
+      <limit effort="1000" lower="${radians(-270)}" upper="${radians(270)}" velocity="${radians(540)}" />
+      <dynamics damping="0.7" friction="0.0"/>
     </joint>
     <!-- joint 5 -->
@@ -179,5 +183,6 @@
       <child link="${prefix}link5" />
       <axis xyz="0 1 0" />
-      <limit effort="0" lower="${radians(-120)}" upper="${radians(120)}" velocity="${radians(540)}" />
+      <limit effort="1000" lower="${radians(-120)}" upper="${radians(120)}" velocity="${radians(540)}" />
+      <dynamics damping="0.7" friction="0.0"/>
     </joint>
     <!-- joint 6 -->
@@ -187,5 +192,6 @@
       <child link="${prefix}link6" />
       <axis xyz="0 0 1" />
-      <limit effort="0" lower="${radians(-360)}" upper="${radians(360)}" velocity="${radians(864)}" />
+      <limit effort="1000" lower="${radians(-360)}" upper="${radians(360)}" velocity="${radians(864)}" />
+      <dynamics damping="0.7" friction="0.0"/>
     </joint>
     <!-- tool frame - fixed frame -->

Commit message: Add fake controller for one side robot control

File: denso_robot_description/urdf/denso_robot.urdf.xacro (robot description, xacro)
@@ -3,7 +3,4 @@
   <!-- Use this if parameters are set from the launch file, otherwise delete -->
   <xacro:arg name="prefix" default="" />
-  <xacro:arg name="sim_gazebo_classic" default="false" />
-  <xacro:arg name="sim_gazebo" default="true" />
-  <xacro:arg name="simulation_controllers" default="" />
   <xacro:arg name="robot_ip" default="192.168.0.1" />
   <xacro:arg name="robot_port" default="5007"/>
@@ -11,4 +8,13 @@
   <xacro:arg name="recv_format" default="292"/>
   <xacro:arg name="config_file" default=""/>
+  <!-- Simulation parameters -->
+  <xacro:arg name="use_fake_hardware" default="false" />
+  <xacro:arg name="fake_sensor_commands" default="false" />
+  <xacro:arg name="sim_gazebo_classic" default="false" />
+  <xacro:arg name="sim_gazebo" default="true" />
+  <!-- initial position for simulations (Fake Hardware, Gazebo, Ignition) -->
+  <xacro:arg name="initial_positions_file" default="$(find denso_robot_description)/config/initial_positions.yaml"/>
+  <!-- convert to property to use substitution in function -->
+  <xacro:property name="initial_positions_file" default="$(arg initial_positions_file)"/>
   <!-- Import Denso Robot Model -->
   <xacro:include filename="$(find denso_robot_description)/urdf/denso_robot/denso_robot_macro.xacro"/>
@@ -29,5 +35,7 @@
     send_format="$(arg send_format)"
     recv_format="$(arg recv_format)"
-    config_file="$(arg config_file)"/>
+    config_file="$(arg config_file)"
+    use_fake_hardware="$(arg use_fake_hardware)"
+    fake_sensor_commands="$(arg fake_sensor_commands)"/>
   <xacro:if value="$(arg sim_gazebo)">
     <gazebo>

File: denso_robot_description/urdf/denso_robot/denso_robot_macro.ros2_control.xacro (robot description, xacro)
@@ -2,4 +2,5 @@
 <robot xmlns:xacro="http://www.ros.org/wiki/xacro">
   <xacro:macro name="denso_robot_ros2_control" params="name prefix
+    use_fake_hardware:=^|false fake_sensor_commands:=^|false
     sim_gazebo_classic:=^|false
     sim_gazebo:=^|true
@@ -18,5 +19,10 @@
           <plugin>gz_ros2_control/GazeboSimSystem</plugin>
         </xacro:if>
-        <xacro:unless value="${sim_gazebo_classic or sim_gazebo}">
+        <xacro:if value="${use_fake_hardware}">
+          <plugin>fake_components/GenericSystem</plugin>
+          <param name="fake_sensor_commands">${fake_sensor_commands}</param>
+          <param name="state_following_offset">0.0</param>
+        <!-- </xacro:if> -->
+        <xacro:unless value="${use_fake_hardware or sim_gazebo_classic or sim_gazebo}">
           <plugin>denso_hw/denso_hw</plugin>
           <param name="robot_ip">${robot_ip}</param>
@@ -33,5 +39,8 @@
           <param name="max">${radians(170)}</param>
         </command_interface>
-        <state_interface name="position"/>
+        <state_interface name="position">
+          <!-- initial position for the FakeSystem and simulation -->
+          <param name="initial_value">0.0</param>
+        </state_interface>/>
         <state_interface name="velocity"/>
         <state_interface name="effort"/>
@@ -42,5 +51,8 @@
           <param name="max">${radians(135)}</param>
         </command_interface>
-        <state_interface name="position"/>
+        <state_interface name="position">
+          <!-- initial position for the FakeSystem and simulation -->
+          <param name="initial_value">0.0</param>
+        </state_interface>/>
         <state_interface name="velocity"/>
         <state_interface name="effort"/>
@@ -51,5 +63,8 @@
           <param name="max">${radians(153)}</param>
         </command_interface>
-        <state_interface name="position"/>
+        <state_interface name="position">
+          <!-- initial position for the FakeSystem and simulation -->
+          <param name="initial_value">1.5708</param>
+        </state_interface>/>
         <state_interface name="velocity"/>
         <state_interface name="effort"/>
@@ -60,5 +75,8 @@
           <param name="max">${radians(270)}</param>
         </command_interface>
-        <state_interface name="position"/>
+        <state_interface name="position">
+          <!-- initial position for the FakeSystem and simulation -->
+          <param name="initial_value">0.0</param>
+        </state_interface>/>
         <state_interface name="velocity"/>
         <state_interface name="effort"/>
@@ -69,5 +87,8 @@
           <param name="max">${radians(120)}</param>
         </command_interface>
-        <state_interface name="position"/>
+        <state_interface name="position">
+          <!-- initial position for the FakeSystem and simulation -->
+          <param name="initial_value">0.0</param>
+        </state_interface>/>
         <state_interface name="velocity"/>
         <state_interface name="effort"/>
@@ -78,5 +99,8 @@
           <param name="max">${radians(360)}</param>
         </command_interface>
-        <state_interface name="position"/>
+        <state_interface name="position">
+          <!-- initial position for the FakeSystem and simulation -->
+          <param name="initial_value">0.0</param>
+        </state_interface>/>
         <state_interface name="velocity"/>
         <state_interface name="effort"/>

Commit message: update fake control

File: denso_robot_description/urdf/denso_robot.urdf.xacro (robot description, xacro)
@@ -3,4 +3,10 @@
   <!-- Use this if parameters are set from the launch file, otherwise delete -->
   <xacro:arg name="prefix" default="" />
+  <!-- Simulation parameters -->
+  <xacro:arg name="use_fake_hardware" default="false" />
+  <xacro:arg name="fake_sensor_commands" default="false" />
+  <xacro:arg name="sim_gazebo_classic" default="false" />
+  <xacro:arg name="sim_gazebo" default="true" />
+  <!-- Real Robot -->
   <xacro:arg name="robot_ip" default="192.168.0.1" />
   <xacro:arg name="robot_port" default="5007"/>
@@ -8,13 +14,4 @@
   <xacro:arg name="recv_format" default="292"/>
   <xacro:arg name="config_file" default=""/>
-  <!-- Simulation parameters -->
-  <xacro:arg name="use_fake_hardware" default="false" />
-  <xacro:arg name="fake_sensor_commands" default="false" />
-  <xacro:arg name="sim_gazebo_classic" default="false" />
-  <xacro:arg name="sim_gazebo" default="true" />
-  <!-- initial position for simulations (Fake Hardware, Gazebo, Ignition) -->
-  <xacro:arg name="initial_positions_file" default="$(find denso_robot_description)/config/initial_positions.yaml"/>
-  <!-- convert to property to use substitution in function -->
-  <xacro:property name="initial_positions_file" default="$(arg initial_positions_file)"/>
   <!-- Import Denso Robot Model -->
   <xacro:include filename="$(find denso_robot_description)/urdf/denso_robot/denso_robot_macro.xacro"/>

Commit message: add initial position for gazebo

File: denso_robot_description/urdf/denso_robot.urdf.xacro (robot description, xacro)
@@ -18,4 +18,8 @@
   <!-- Import ROS2 Control -->
   <xacro:include filename="$(find denso_robot_description)/urdf/denso_robot/denso_robot_macro.ros2_control.xacro"/>
+  <!-- initial position for simulations (Fake Hardware, Gazebo, Ignition) -->
+  <xacro:arg name="initial_positions_file" default="$(find denso_robot_description)/config/initial_positions.yaml"/>
+  <!-- convert to property to use substitution in function -->
+  <xacro:property name="initial_positions_file" default="$(arg initial_positions_file)"/>
   <!-- create link fixed to the "world" -->
   <link name="world" />
@@ -34,5 +38,6 @@
     config_file="$(arg config_file)"
     use_fake_hardware="$(arg use_fake_hardware)"
-    fake_sensor_commands="$(arg fake_sensor_commands)"/>
+    fake_sensor_commands="$(arg fake_sensor_commands)"
+    initial_positions="${xacro.load_yaml(initial_positions_file)}"/>
   <xacro:if value="$(arg sim_gazebo)">
     <gazebo>

File: denso_robot_description/urdf/denso_robot/denso_robot_macro.ros2_control.xacro (robot description, xacro)
@@ -10,5 +10,6 @@
     recv_format
     controller_type:=^|8
-    config_file ">
+    config_file
+    initial_positions:=${dict(joint1=0.0,joint2=0.0,joint3=1.57,joint4=0.0,joint5=0.0,joint6=0.0)}">
     <ros2_control name="${name}" type="system">
       <hardware>
@@ -41,6 +42,6 @@
         <state_interface name="position">
           <!-- initial position for the FakeSystem and simulation -->
-          <param name="initial_value">0.0</param>
-        </state_interface>/>
+          <param name="initial_value">${initial_positions['joint1']}</param>
+        </state_interface>
         <state_interface name="velocity"/>
         <state_interface name="effort"/>
@@ -53,6 +54,6 @@
         <state_interface name="position">
           <!-- initial position for the FakeSystem and simulation -->
-          <param name="initial_value">0.0</param>
-        </state_interface>/>
+          <param name="initial_value">${initial_positions['joint2']}</param>
+        </state_interface>
         <state_interface name="velocity"/>
         <state_interface name="effort"/>
@@ -65,6 +66,6 @@
         <state_interface name="position">
           <!-- initial position for the FakeSystem and simulation -->
-          <param name="initial_value">1.5708</param>
-        </state_interface>/>
+          <param name="initial_value">${initial_positions['joint3']}</param>
+        </state_interface>
         <state_interface name="velocity"/>
         <state_interface name="effort"/>
@@ -77,6 +78,6 @@
         <state_interface name="position">
           <!-- initial position for the FakeSystem and simulation -->
-          <param name="initial_value">0.0</param>
-        </state_interface>/>
+          <param name="initial_value">${initial_positions['joint4']}</param>
+        </state_interface>
         <state_interface name="velocity"/>
         <state_interface name="effort"/>
@@ -89,6 +90,6 @@
         <state_interface name="position">
           <!-- initial position for the FakeSystem and simulation -->
-          <param name="initial_value">0.0</param>
-        </state_interface>/>
+          <param name="initial_value">${initial_positions['joint5']}</param>
+        </state_interface>
         <state_interface name="velocity"/>
         <state_interface name="effort"/>
@@ -101,6 +102,6 @@
         <state_interface name="position">
           <!-- initial position for the FakeSystem and simulation -->
-          <param name="initial_value">0.0</param>
-        </state_interface>/>
+          <param name="initial_value">${initial_positions['joint6']}</param>
+        </state_interface>
         <state_interface name="velocity"/>
         <state_interface name="effort"/>

File: denso_robot_description/urdf/denso_robot/denso_robot_macro.xacro (robot description, xacro)
@@ -2,5 +2,10 @@
 <robot xmlns:xacro="http://wiki.ros.org/xacro">
   <xacro:include filename="$(find denso_robot_description)/urdf/common.xacro" />
-  <xacro:macro name="denso_robot" params="prefix parent *origin">
+  <xacro:macro name="denso_robot" params="
+    prefix
+    parent
+    *origin
+    initial_positions:=${dict(joint1=0.0,joint2=0.0,joint3=1.57,joint4=0.0,joint5=0.0,joint6=0.0)}"
+    >
     <!-- LINKS -->
     <!-- base link -->
